File: kicad/acoustic_transmitter.kicad_sch (KiCad schematic)
At the start: 28 parts, among them Q1 IRF6613, Q2 IRF6613, U1 LM311, U2 LM358, U3 LM358, U4 LM358, U5 class AB, U6 IR2110, U7 74HC14, U8 MCP4822

Commit message: add virtual ground and star routing
Parts:
- added C1, C4, C5: C_US, symbol Device:C_US
- added R13: R, symbol Device:R
- U2: value LM358 -> NJM2137D
Connections:
- net +15V is gone; now on net +5V: U1.8 (V+)
- net -VBUS is gone; now on net GND: Q2.3 (S)
- net +12V: now also C1.1, C4.1, C5.1; no longer U6.3 (VCC)
- net at D1.1 (K), D2.2 (A): now also R13.2; no longer R12.2
- net +5V: now reaches U6.9 (VDD)
- net VBUS: no longer names the net of Q1.1 (D)
- net VBUS: now also C4.2
- new net: C1.2, C5.2, U6.3 (VCC)
- new net: R12.2, R13.1
- no-connect marks 0 -> 1
Other:
- note added: "-VBUS"
- note added: "VBUS"
- note added: "bulk power"
- note added: "hex inverter square signal and clean"
- note added: "integrator"
- note added: "level shifting"
- note added: "square wave Schmitt Trigger"
- moved on the sheet: BZ1, D1, D2, Q1, Q2, R10, R12, R8, R9, U6, U7A
